File: pcb/keyboard_pcb-rounded.kicad_pcb (KiCad board)
At the start: 2 copper layers, 138.8 x 89.9 mm, 23 parts, among them J1 TRRS, K00 KEYSW, K01 KEYSW, K02 KEYSW, K03 KEYSW, K04 KEYSW, K05 KEYSW, K10 KEYSW, K11 KEYSW, K12 KEYSW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

Commit message: Add holes for the brass standoffs
Parts:
- added H1: MountingHole, cantor:Standoff_Hole, F.Cu at (83.0, 78.5)
- added H2: MountingHole, cantor:Standoff_Hole, F.Cu at (155.0, 67.6)
- added H3: MountingHole, cantor:Standoff_Hole, F.Cu at (83.0, 95.5)
- added H4: MountingHole, cantor:Standoff_Hole, F.Cu at (173.9, 116.4)
Routing:
- net +3V3: track 45.1 -> 91.8 mm
- net GND: track 608.5 -> 567.2 mm
- net /k00: track 163.8 -> 136.1 mm, vias 1 -> 0
- net /k25: track 87.2 -> 82.0 mm
- net /k02: track 94.6 -> 95.8 mm
- net /k04: track 58.0 -> 59.1 mm
- net /k03: track 76.3 -> 77.4 mm
- net /k01: track 116.8 -> 117.9 mm
Other:
- board text added: "Cantor rev1.1"
- board text removed: "Cantor rev1.0"
