File: pcb/keyboard_pcb.kicad_sch (KiCad schematic)
At the start: 23 parts, among them J1 TRRS, K00 KEYSW, K01 KEYSW, K02 KEYSW, K03 KEYSW, K04 KEYSW, K05 KEYSW, K10 KEYSW, K11 KEYSW, K12 KEYSW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

Commit message: Add holes for the brass standoffs
Parts:
- added H1, H2, H3, H4: MountingHole, cantor:Standoff_Hole, symbol Mechanical:MountingHole
Changed lines of the file:
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@@
     (pin "2")
+  )
+  (symbol (lib_id "Mechanical:MountingHole") (at 50.165 147.955 0) (unit 1)
+    (in_bom yes) (on_board yes) (fields_autoplaced)
+    (property "Reference" "H3" (id 0) (at 53.34 146.6849 0)
+      (effects (font (size 1.27 1.27)) (justify left))
+    )
+    (property "Value" "MountingHole" (id 1) (at 53.34 149.2249 0)
+      (effects (font (size 1.27 1.27)) (justify left))
+    )
+    (property "Footprint" "cantor:Standoff_Hole" (id 2) (at 50.165 147.955 0)
+      (effects (font (size 1.27 1.27)) hide)
+    )
+    (property "Datasheet" "~" (id 3) (at 50.165 147.955 0)
+      (effects (font (size 1.27 1.27)) hide)
+    )
   )
   (symbol (lib_id "power:GND") (at 64.77 125.73 0) (unit 1)
@@
   (symbol (lib_id "power:+3V3") (at 64.77 118.11 0) (unit 1)
     (in_bom yes) (on_board yes) (fields_autoplaced)
-    (property "Reference" "#PWR?" (id 0) (at 64.77 121.92 0)
+    (property "Reference" "#PWR0127" (id 0) (at 64.77 121.92 0)
       (effects (font (size 1.27 1.27)) hide)
     )
@@
     (pin "1")
   )
+  (symbol (lib_id "Mechanical:MountingHole") (at 50.165 142.875 0) (unit 1)
+    (in_bom yes) (on_board yes) (fields_autoplaced)
+    (property "Reference" "H1" (id 0) (at 53.34 141.6049 0)
+      (effects (font (size 1.27 1.27)) (justify left))
+    )
+    (property "Value" "MountingHole" (id 1) (at 53.34 144.1449 0)
+      (effects (font (size 1.27 1.27)) (justify left))
+    )
+    (property "Footprint" "cantor:Standoff_Hole" (id 2) (at 50.165 142.875 0)
+      (effects (font (size 1.27 1.27)) hide)
+    )
+    (property "Datasheet" "~" (id 3) (at 50.165 142.875 0)
+      (effects (font (size 1.27 1.27)) hide)
+    )
+  )
   (symbol (lib_id "keyboard_parts:KEYSW") (at 213.36 60.96 0) (mirror y) (unit 1)
     (in_bom yes) (on_board yes)
@@
     (pin "1")
     (pin "2")
+  )
+  (symbol (lib_id "Mechanical:MountingHole") (at 70.485 142.875 0) (unit 1)
+    (in_bom yes) (on_board yes) (fields_autoplaced)
+    (property "Reference" "H2" (id 0) (at 73.66 141.6049 0)
+      (effects (font (size 1.27 1.27)) (justify left))
+    )
+    (property "Value" "MountingHole" (id 1) (at 73.66 144.1449 0)
+      (effects (font (size 1.27 1.27)) (justify left))
+    )
+    (property "Footprint" "cantor:Standoff_Hole" (id 2) (at 70.485 142.875 0)
+      (effects (font (size 1.27 1.27)) hide)
+    )
+    (property "Datasheet" "~" (id 3) (at 70.485 142.875 0)
+      (effects (font (size 1.27 1.27)) hide)
+    )
   )
   (symbol (lib_id "power:GND") (at 220.98 33.02 0) (unit 1)
@@
   (symbol (lib_id "power:+3V3") (at 44.45 87.63 0) (unit 1)
     (in_bom yes) (on_board yes) (fields_autoplaced)
-    (property "Reference" "#PWR?" (id 0) (at 44.45 91.44 0)
+    (property "Reference" "#PWR0125" (id 0) (at 44.45 91.44 0)
       (effects (font (size 1.27 1.27)) hide)
     )
@@
   (symbol (lib_id "power:+3V3") (at 104.14 39.37 0) (unit 1)
     (in_bom yes) (on_board yes) (fields_autoplaced)
-    (property "Reference" "#PWR?" (id 0) (at 104.14 43.18 0)
+    (property "Reference" "#PWR0111" (id 0) (at 104.14 43.18 0)
       (effects (font (size 1.27 1.27)) hide)
     )
@@
     )
     (pin "1")
+  )
+  (symbol (lib_id "Mechanical:MountingHole") (at 70.485 147.955 0) (unit 1)
+    (in_bom yes) (on_board yes) (fields_autoplaced)
+    (property "Reference" "H4" (id 0) (at 73.66 146.6849 0)
+      (effects (font (size 1.27 1.27)) (justify left))
+    )
+    (property "Value" "MountingHole" (id 1) (at 73.66 149.2249 0)
+      (effects (font (size 1.27 1.27)) (justify left))
+    )
+    (property "Footprint" "cantor:Standoff_Hole" (id 2) (at 70.485 147.955 0)
+      (effects (font (size 1.27 1.27)) hide)
+    )
+    (property "Datasheet" "~" (id 3) (at 70.485 147.955 0)
+      (effects (font (size 1.27 1.27)) hide)
+    )
   )
   (symbol (lib_id "keyboard_parts:KEYSW") (at 264.16 30.48 0) (mirror y) (unit 1)
@@
       (reference "#PWR0110") (unit 1) (value "GND") (footprint "")
     )
+    (path "/dca1eae4-b54a-457a-98d3-85f0bf91ed0c"
+      (reference "#PWR0111") (unit 1) (value "+3V3") (footprint "")
+    )
     (path "/808eaac8-875a-4854-a593-0732e2dcbd2c"
       (reference "#PWR0112") (unit 1) (value "GND") (footprint "")
@@
       (reference "#PWR0124") (unit 1) (value "GND") (footprint "")
     )
+    (path "/cc6043c3-0bcf-4511-9f1f-e76c5c60bcaa"
+      (reference "#PWR0125") (unit 1) (value "+3V3") (footprint "")
+    )
     (path "/284bc30d-04b3-44eb-8dce-848f7e5cb450"
       (reference "#PWR0126") (unit 1) (value "GND") (footprint "")
     )
     (path "/778761f4-c241-4a95-8ab0-2cd0f571f8b7"
-      (reference "#PWR?") (unit 1) (value "+3V3") (footprint "")
-    )
-    (path "/cc6043c3-0bcf-4511-9f1f-e76c5c60bcaa"
-      (reference "#PWR?") (unit 1) (value "+3V3") (footprint "")
-    )
-    (path "/dca1eae4-b54a-457a-98d3-85f0bf91ed0c"
-      (reference "#PWR?") (unit 1) (value "+3V3") (footprint "")
+      (reference "#PWR0127") (unit 1) (value "+3V3") (footprint "")
+    )
+    (path "/a7900784-bc94-484c-8e21-637a65966b52"
+      (reference "H1") (unit 1) (value "MountingHole") (footprint "cantor:Standoff_Hole")
+    )
+    (path "/c2fc87dc-6ac6-40e4-ad37-eb3538b51316"
+      (reference "H2") (unit 1) (value "MountingHole") (footprint "cantor:Standoff_Hole")
+    )
+    (path "/26d24eef-b4df-46dc-a93c-d2fc6e635995"
+      (reference "H3") (unit 1) (value "MountingHole") (footprint "cantor:Standoff_Hole")
+    )
+    (path "/fb47ff47-d1ba-49ec-90e8-9f5bb92644fd"
+      (reference "H4") (unit 1) (value "MountingHole") (footprint "cantor:Standoff_Hole")
     )
     (path "/8901fa8c-a4aa-47e4-b9d5-827b4e7d5c4d"
